File: Non-Detachable-Without-GPS/RFM_STM_Breakout.kicad_sch (KiCad schematic)
At the start: 29 parts, among them J1 USB_B_Micro, J2 Conn_01x02_Male, J3 Conn_01x16_Male, J4 Conn_01x12_Male, J5 Conn_01x15_Male, J6 Conn_Coaxial, SW1 SW_Push, U1 RFM95W-868S2, U2 XC6206P332MR, U3 STM32L053R8Tx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

Commit message: Update USB Pullup (R already internal in STM32L0 processors)
Parts:
- removed R3: 1k5, Resistor_SMD:R_0603_1608Metric, symbol Device:R_Small
Changed lines of the file:
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@@
   (junction (at 21.59 69.85) (diameter 0) (color 0 0 0 0)
-  )
-  (junction (at 266.7 81.28) (diameter 0) (color 0 0 0 0)
   )
   (junction (at 231.14 137.16) (diameter 0) (color 0 0 0 0)
@@
     (stroke (width 0) (type default) (color 0 0 0 0))
   )
-  (wire (pts (xy 266.7 76.2) (xy 266.7 81.28))
-    (stroke (width 0) (type default) (color 0 0 0 0))
-  )
   (wire (pts (xy 241.3 45.72) (xy 246.38 45.72))
     (stroke (width 0) (type default) (color 0 0 0 0))
@@
     (stroke (width 0) (type default) (color 0 0 0 0))
   )
-  (wire (pts (xy 251.46 81.28) (xy 266.7 81.28))
+  (wire (pts (xy 251.46 81.28) (xy 267.97 81.28))
     (stroke (width 0) (type default) (color 0 0 0 0))
   )
@@
   )
   (wire (pts (xy 52.07 76.2) (xy 52.07 77.47))
-    (stroke (width 0) (type default) (color 0 0 0 0))
-  )
-  (wire (pts (xy 267.97 81.28) (xy 266.7 81.28))
     (stroke (width 0) (type default) (color 0 0 0 0))
   )
@@
     )
     (property "Datasheet" "" (id 3) (at 157.48 182.88 0)
-      (effects (font (size 1.27 1.27)) hide)
-    )
-    (pin "1")
-  )
-  (symbol (lib_id "power:+3.3V") (at 266.7 71.12 0) (unit 1)
-    (in_bom yes) (on_board yes)
-    (property "Reference" "#PWR0110" (id 0) (at 266.7 74.93 0)
-      (effects (font (size 1.27 1.27)) hide)
-    )
-    (property "Value" "+3.3V" (id 1) (at 266.7 67.31 0))
-    (property "Footprint" "" (id 2) (at 266.7 71.12 0)
-      (effects (font (size 1.27 1.27)) hide)
-    )
-    (property "Datasheet" "" (id 3) (at 266.7 71.12 0)
       (effects (font (size 1.27 1.27)) hide)
     )
@@
     (pin "2")
   )
-  (symbol (lib_id "Device:R_Small") (at 266.7 73.66 0) (unit 1)
-    (in_bom yes) (on_board yes)
-    (property "Reference" "R3" (id 0) (at 268.1986 72.4916 0)
-      (effects (font (size 1.27 1.27)) (justify left))
-    )
-    (property "Value" "1k5" (id 1) (at 268.1986 74.803 0)
-      (effects (font (size 1.27 1.27)) (justify left))
-    )
-    (property "Footprint" "Resistor_SMD:R_0603_1608Metric" (id 2) (at 266.7 73.66 0)
-      (effects (font (size 1.27 1.27)) hide)
-    )
-    (property "Datasheet" "~" (id 3) (at 266.7 73.66 0)
-      (effects (font (size 1.27 1.27)) hide)
-    )
-    (property "LCSC Part #" "C22842" (id 4) (at 266.7 73.66 0)
-      (effects (font (size 1.27 1.27)) hide)
-    )
-    (pin "1")
-    (pin "2")
-  )
   (symbol (lib_id "power:GND") (at 209.55 43.18 0) (unit 1)
     (in_bom yes) (on_board yes)
@@
       (reference "#PWR0109") (unit 1) (value "GND") (footprint "")
     )
-    (path "/18b7848b-3271-46c5-a425-a96f6e85b251"
-      (reference "#PWR0110") (unit 1) (value "+3.3V") (footprint "")
-    )
     (path "/39a1d3de-e80c-4990-9d87-c6cb905fae7c"
       (reference "#PWR0111") (unit 1) (value "+3.3V") (footprint "")
@@
       (reference "R2") (unit 1) (value "10k") (footprint "Resistor_SMD:R_0603_1608Metric")
     )
-    (path "/f0b512f0-3c35-4ac7-8f2d-ff9535d072b0"
-      (reference "R3") (unit 1) (value "1k5") (footprint "Resistor_SMD:R_0603_1608Metric")
-    )
     (path "/234d3392-03df-437c-8ca8-ff48e85c0c95"
